Commit message: fix(description): remove legacy padding and duplicate fixed gripper

File: src/chess_robot_description/urdf/nova5_with_ag95.urdf (robot description, URDF)
Before this commit: robot nova5_with_ag95, 21 links, 20 joints
Links:
- removed link safety_padding_link
- link camera_bracket_link: geometry collision mesh filename=package://chess_robot_description/meshes/tool_mount/camera_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; visual mesh filename=package://chess_robot_description/meshes/tool_mount/camera_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
- link left_finger: geometry collision mesh filename=package://dh_ag95_description/meshes/collision/finger.stl scale=0.001 0.001 0.001; visual mesh filename=package://dh_ag95_description/meshes/visual/finger.stl scale=0.001 0.001 0.001
- link left_finger_pad: geometry collision mesh filename=package://dh_ag95_description/meshes/collision/finger_pad.s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 scale=0.001 0.001 0.001; visual mesh filename=package://dh_ag95_description/meshes/visual/finger_pad.stl scale=0.001 0.001 0.001
- link right_finger: geometry collision mesh filename=package://dh_ag95_description/meshes/collision/finger.stl scale=0.001 0.001 0.001; visual mesh filename=package://dh_ag95_description/meshes/visual/finger.stl scale=0.001 0.001 0.001
- link right_finger_pad: geometry collision mesh filename=package://dh_ag95_description/meshes/collision/finger_pad.s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 scale=0.001 0.001 0.001; visual mesh filename=package://dh_ag95_description/meshes/visual/finger_pad.stl scale=0.001 0.001 0.001
Joints:
- removed joint safety_padding_joint
- joint left_finger_joint: limit lower=-0.01 upper=1.11 effort=50.0 velocity=2.1 -> lower=-0.01 upper=0.95 effort=50.0 velocity=2.1
- joint left_inner_knuckle_joint: limit lower=-0.01 upper=1.11 effort=50.0 velocity=2.1 -> lower=-0.01 upper=0.95 effort=50.0 velocity=2.1
- joint left_outer_knuckle_joint: limit lower=0.0 upper=1.1 effort=50.0 velocity=2.1 -> lower=0.0 upper=0.94 effort=50.0 velocity=2.1
- joint right_finger_joint: limit lower=-0.01 upper=1.11 effort=50.0 velocity=2.1 -> lower=-0.01 upper=0.95 effort=50.0 velocity=2.1
- joint right_inner_knuckle_joint: limit lower=-0.01 upper=1.11 effort=50.0 velocity=2.1 -> lower=-0.01 upper=0.95 effort=50.0 velocity=2.1
- joint right_outer_knuckle_joint: limit lower=-0.01 upper=1.11 effort=50.0 velocity=2.1 -> lower=-0.01 upper=0.95 effort=50.0 velocity=2.1

File: src/chess_robot_description/urdf/nova5_with_ag95.urdf.xacro (robot description, xacro)
@@ -6,18 +6,22 @@
   <xacro:include filename="$(arg ag95_macro_file)"/>
   <xacro:arg name="include_ground" default="false"/>
-  <xacro:arg name="include_legacy_padding" default="true"/>
-  <!-- Legacy mounting geometry and transforms; not a new calibration. -->
+  <!-- Unmeasured calibration defaults; model changes do not move hardware. -->
+  <xacro:arg name="gripper_mount_z" default="0.0085"/>
+  <xacro:arg name="grasp_link_offset" default="0.20"/>
+  <xacro:arg name="gripper_joint_upper_limit" default="0.94"/>
+  <!-- Rear camera and mounting components only; original composite also contained
+       a complete fixed AG95, which must not duplicate the articulated gripper. -->
   <link name="camera_bracket_link">
     <visual>
-      <origin xyz="0.09419 -0.10218 0.18445" rpy="0 3.14159 0"/>
+      <origin xyz="0 0 0" rpy="0 0 0"/>
       <geometry>
-        <mesh filename="package://chess_robot_description/meshes/tool_mount/new_jiazhua1.STL" scale="0.001 0.001 0.001"/>
+        <mesh filename="package://chess_robot_description/meshes/tool_mount/camera_mount_assembly_m.stl"/>
       </geometry>
       <material name="silver"><color rgba="0.75 0.75 0.75 1.0"/></material>
     </visual>
     <collision>
-      <origin xyz="0.09419 -0.10218 0.18445" rpy="0 3.14159 0"/>
+      <origin xyz="0 0 0" rpy="0 0 0"/>
       <geometry>
-        <mesh filename="package://chess_robot_description/meshes/tool_mount/new_jiazhua1.STL" scale="0.001 0.001 0.001"/>
+        <mesh filename="package://chess_robot_description/meshes/tool_mount/camera_mount_assembly_m.stl"/>
       </geometry>
     </collision>
@@ -28,26 +32,9 @@
     <origin xyz="0 0 0" rpy="0 0 0"/>
   </joint>
-  <xacro:dh_ag95_gripper prefix="" parent="camera_bracket_link" grasp_link_offset="0.20">
-    <origin xyz="0 0 0.0085" rpy="0 0 0"/>
+  <xacro:dh_ag95_gripper prefix="" parent="camera_bracket_link"
+      grasp_link_offset="$(arg grasp_link_offset)"
+      joint_upper_limit="$(arg gripper_joint_upper_limit)">
+    <origin xyz="0 0 $(arg gripper_mount_z)" rpy="0 0 0"/>
   </xacro:dh_ag95_gripper>
-  <!-- Preserve the old extra collision envelope, independently switchable. -->
-  <xacro:if value="$(arg include_legacy_padding)">
-    <link name="safety_padding_link">
-      <visual>
-        <origin xyz="0 0.0305 0.0825" rpy="0 0 0"/>
-        <geometry><box size="0.115 0.001 0.165"/></geometry>
-        <material name="blue"><color rgba="0.0 0.0 1.0 0.6"/></material>
-      </visual>
-      <collision>
-        <origin xyz="0 0.0305 0.0825" rpy="0 0 0"/>
-        <geometry><box size="0.115 0.001 0.165"/></geometry>
-      </collision>
-    </link>
-    <joint name="safety_padding_joint" type="fixed">
-      <parent link="ag95_base_link"/>
-      <child link="safety_padding_link"/>
-      <origin xyz="0 0 0" rpy="0 0 0"/>
-    </joint>
-  </xacro:if>
   <!-- Scene geometry is optional; not part of the default robot model. -->
   <xacro:if value="$(arg include_ground)">

File: src/dh_ag95_description/urdf/ag95.urdf (robot description, URDF)
Before this commit: robot ag95_preview, 12 links, 11 joints
Links:
- link left_finger: geometry collision mesh filename=package://dh_ag95_description/meshes/collision/finger.stl scale=0.001 0.001 0.001; visual mesh filename=package://dh_ag95_description/meshes/visual/finger.stl scale=0.001 0.001 0.001
- link left_finger_pad: geometry collision mesh filename=package://dh_ag95_description/meshes/collision/finger_pad.s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 scale=0.001 0.001 0.001; visual mesh filename=package://dh_ag95_description/meshes/visual/finger_pad.stl scale=0.001 0.001 0.001
- link right_finger: geometry collision mesh filename=package://dh_ag95_description/meshes/collision/finger.stl scale=0.001 0.001 0.001; visual mesh filename=package://dh_ag95_description/meshes/visual/finger.stl scale=0.001 0.001 0.001
- link right_finger_pad: geometry collision mesh filename=package://dh_ag95_description/meshes/collision/finger_pad.s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 scale=0.001 0.001 0.001; visual mesh filename=package://dh_ag95_description/meshes/visual/finger_pad.stl scale=0.001 0.001 0.001
Joints:
- joint left_finger_joint: limit lower=-0.01 upper=1.11 effort=50.0 velocity=2.1 -> lower=-0.01 upper=0.95 effort=50.0 velocity=2.1
- joint left_inner_knuckle_joint: limit lower=-0.01 upper=1.11 effort=50.0 velocity=2.1 -> lower=-0.01 upper=0.95 effort=50.0 velocity=2.1
- joint left_outer_knuckle_joint: limit lower=0.0 upper=1.1 effort=50.0 velocity=2.1 -> lower=0.0 upper=0.94 effort=50.0 velocity=2.1
- joint right_finger_joint: limit lower=-0.01 upper=1.11 effort=50.0 velocity=2.1 -> lower=-0.01 upper=0.95 effort=50.0 velocity=2.1
- joint right_inner_knuckle_joint: limit lower=-0.01 upper=1.11 effort=50.0 velocity=2.1 -> lower=-0.01 upper=0.95 effort=50.0 velocity=2.1
- joint right_outer_knuckle_joint: limit lower=-0.01 upper=1.11 effort=50.0 velocity=2.1 -> lower=-0.01 upper=0.95 effort=50.0 velocity=2.1

File: src/dh_ag95_description/urdf/ag95.urdf.xacro (robot description, xacro)
@@ -4,5 +4,9 @@
   <xacro:include filename="dh_ag95_macro.xacro"/>
   <link name="world"/>
-  <xacro:dh_ag95_gripper prefix="" parent="world" grasp_link_offset="0.20">
+  <xacro:arg name="gripper_joint_upper_limit" default="0.94"/>
+  <xacro:arg name="grasp_link_offset" default="0.20"/>
+  <xacro:dh_ag95_gripper prefix="" parent="world"
+      grasp_link_offset="$(arg grasp_link_offset)"
+      joint_upper_limit="$(arg gripper_joint_upper_limit)">
     <origin xyz="0 0 0" rpy="0 0 0"/>
   </xacro:dh_ag95_gripper>

File: src/dh_ag95_description/urdf/dh_ag95_macro.xacro (robot description, xacro)
@@ -6,9 +6,11 @@
     grasp_link_offset:=0.19
     parent
+    joint_upper_limit:=0.94
     *origin"
   >
-    <!-- this URDF is overly complicated IMO don't bother trying to understand it lol -->
+    <!-- Adapted 2026-10-24: remove legacy collision boxes and expose a geometry-only
+         closing limit. The unmodified source is in reference/ag95/. -->
     <xacro:property name="lower_limit" value="0.0" />
-    <xacro:property name="upper_limit" value="1.10" />
+    <xacro:property name="upper_limit" value="${joint_upper_limit}" />
     <xacro:property name="max_effort" value="50.0" />
     <xacro:property name="max_velocity" value="2.1" />
@@ -105,11 +107,4 @@
           </geometry>
         </collision>
-        <!-- Added 1cm thickness padding block around the finger -->
-        <collision>
-          <origin xyz="-0.0103 0.00875 0.0166" rpy="0 0 0" />
-          <geometry>
-            <box size="0.052 0.041 0.064" />
-          </geometry>
-        </collision>
       </link>
     </xacro:macro>
@@ -143,11 +138,4 @@
             <mesh filename="package://dh_ag95_description/meshes/collision/finger_pad.stl"
               scale="0.001 0.001 0.001" />
-          </geometry>
-        </collision>
-        <!-- Added 1cm thickness padding block around the finger pad -->
-        <collision>
-          <origin xyz="-0.001 0.0 0.0082" rpy="0 0 0" />
-          <geometry>
-            <box size="0.032 0.041 0.054" />
           </geometry>
         </collision>

Commit message: fix(description): install updated user camera fixture

File: src/chess_robot_description/urdf/nova5_with_ag95.urdf (robot description, URDF)
Before this commit: robot nova5_with_ag95, 20 links, 19 joints
Links:
- link ag95_base_link: geometry 
Joints:
- joint gripper_base_joint: origin xyz=0 0 0.0085 rpy=0 0 0 -> xyz=0 0 0.0 rpy=0 0 0

File: src/chess_robot_description/urdf/nova5_with_ag95.urdf.xacro (robot description, xacro)
@@ -6,10 +6,11 @@
   <xacro:include filename="$(arg ag95_macro_file)"/>
   <xacro:arg name="include_ground" default="false"/>
-  <!-- Unmeasured calibration defaults; model changes do not move hardware. -->
-  <xacro:arg name="gripper_mount_z" default="0.0085"/>
+  <!-- New fixture includes the slotted gripper base; flange datums coincide in CAD.
+       Additional mount Z remains adjustable for later physical calibration. -->
+  <xacro:arg name="gripper_mount_z" default="0.0"/>
   <xacro:arg name="grasp_link_offset" default="0.20"/>
   <xacro:arg name="gripper_joint_upper_limit" default="0.94"/>
-  <!-- Rear camera and mounting components only; original composite also contained
-       a complete fixed AG95, which must not duplicate the articulated gripper. -->
+  <!-- User 20260117 v2 fixture: mounting plate, slotted clamp and new camera.
+       Includes the base shape, so the generic AG95 base geometry is omitted below. -->
   <link name="camera_bracket_link">
     <visual>
@@ -34,4 +35,5 @@
   <xacro:dh_ag95_gripper prefix="" parent="camera_bracket_link"
       grasp_link_offset="$(arg grasp_link_offset)"
+      include_base_geometry="false"
       joint_upper_limit="$(arg gripper_joint_upper_limit)">
     <origin xyz="0 0 $(arg gripper_mount_z)" rpy="0 0 0"/>

File: src/dh_ag95_description/urdf/dh_ag95_macro.xacro (robot description, xacro)
@@ -7,4 +7,5 @@
     parent
     joint_upper_limit:=0.94
+    include_base_geometry:=true
     *origin"
   >
@@ -214,21 +215,23 @@
         <inertia ixx="${4e-05*0.291227699}" iyy="${0.000121*0.291227699}" izz="${0.000158*0.291227699}" ixy="${0.0*0.291227699}" iyz="${0.0*0.291227699}" ixz="${-0.0*0.291227699}" />
       </inertial>
-      <visual>
-        <origin xyz="0 0 0" rpy="0 0 0" />
-        <geometry>
-          <mesh filename="package://dh_ag95_description/meshes/visual/base_link.stl"
-            scale="0.001 0.001 0.001" />
-        </geometry>
-        <material name="">
-          <color rgba="0.792156862745098 0.819607843137255 0.933333333333333 1" />
-        </material>
-      </visual>
-      <collision>
-        <origin xyz="0 0 0" rpy="0 0 0" />
-        <geometry>
-          <mesh filename="package://dh_ag95_description/meshes/collision/base_link.stl"
-            scale="0.001 0.001 0.001" />
-        </geometry>
-      </collision>
+      <xacro:if value="${include_base_geometry}">
+        <visual>
+          <origin xyz="0 0 0" rpy="0 0 0" />
+          <geometry>
+            <mesh filename="package://dh_ag95_description/meshes/visual/base_link.stl"
+              scale="0.001 0.001 0.001" />
+          </geometry>
+          <material name="">
+            <color rgba="0.792156862745098 0.819607843137255 0.933333333333333 1" />
+          </material>
+        </visual>
+        <collision>
+          <origin xyz="0 0 0" rpy="0 0 0" />
+          <geometry>
+            <mesh filename="package://dh_ag95_description/meshes/collision/base_link.stl"
+              scale="0.001 0.001 0.001" />
+          </geometry>
+        </collision>
+      </xacro:if>
     </link>
     <!-- main body of gripper -->
